File: led-controller-wrover32.kicad_pcb (KiCad board)
At the start: 4 copper layers, 36 x 40 mm, 135 parts, among them J101 Molex PicoBlade 4-pin, J102 Molex PicoBlade 6-pin, J103 STATUS OUT, J104 USB_B_Micro, J105 POWER IN, J106 Molex PicoBlade 6-pin, J107 5V_LOGIC, J201 12V_OUT, J301 Micro_SD_Card, J302 Molex PicoBlade 4-pin, J401 Fan PWM, J402 GPIO_CONN, Q101 UMH3N, Q301 BSS138, Q401 SIL2301-TP, Q402 EM6K7T2R, SW301 KMR2, SW302 KMR2, U101 TPS2001DDBVX, U102 USBUF02W6, U103 ESP32-S3-WROOM-2-N32R8, U104 NTS0104BQ,115, U201 TPS61089RNRR, U202 MPM3810GQB-33, U301 SSM2518CPZ, U401 SN74AUP1G08YZP, U402 BME280, U403 BNO085, U404 SX1509BIULTRT, Y401 OM-7604-C7

Commit message: Minor fixes.
Signed-off-by: Aaron Williams <aaron.w2@gmail.com>
Parts:
- added TP401: ~{BNO_RST}, TestPoint:TestPoint_Pad_1.0x1.0mm, B.Cu at (90.1, 31.0)
- Q301: value BSS138 -> BSS138PW,115
Routing:
- net /Motion and GPIO/~{BNO085_RST}: track 19.8 -> 20.7 mm
- net GND: track 69.8 -> 69.3 mm, vias 183 -> 181
