File: Motion GPIO.kicad_sch (KiCad schematic)
At the start: 37 parts, among them J111 Fan PWM, J112 GPIO_CONN, Q103 IRFHS9351, Q104 BSS138PW,115, U108 SN74AUP1G08YZP, U109 BME280, U110 BNO086, U111 SX1509BIULTRT, Y101 OM-7604-C7

Commit message: Changed ESP32 to ESP32-S3-WROOM-1 and other cleanup
Signed-off-by: Aaron Williams <aaron.w2@gmail.com>
Parts:
- U108: MFR (none) -> Texas Instruments; MPN (none) -> BQ25180YBGR; SPN (none) -> 296-BQ25180YBGRCT-ND; SPR (none) -> Digikey; SPURL (none) -> https://www.digikey.com/en/products/detail/texas-instrument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
Changed lines of the file:
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@@
   (title_block
     (title "Wroom32 LED Controller")
-    (date "2022-12-02")
+    (date "2022-12-06")
     (rev "4.0.0")
     (company "Aaron Williams")
@@
       (effects (font (size 1.27 1.27)) hide)
     )
+    (property "MFR" "Texas Instruments" (id 5) (at 49.53 30.48 0)
+      (effects (font (size 1.27 1.27)) hide)
+    )
+    (property "MPN" "BQ25180YBGR" (id 6) (at 49.53 30.48 0)
+      (effects (font (size 1.27 1.27)) hide)
+    )
+    (property "SPN" "296-BQ25180YBGRCT-ND" (id 7) (at 49.53 30.48 0)
+      (effects (font (size 1.27 1.27)) hide)
+    )
+    (property "SPR" "Digikey" (id 8) (at 49.53 30.48 0)
+      (effects (font (size 1.27 1.27)) hide)
+    )
+    (property "SPURL" "https://www.digikey.com/en/products/detail/texas-instruments/BQ25180YBGR/15857374" (id 9) (at 49.53 30.48 0)
+      (effects (font (size 1.27 1.27)) hide)
+    )
